File: 3PDT Board wLED.brd (EAGLE design)
At the start: 29.6 x 23.5 mm, 11 parts, among them SW2 3PDT

Commit message: Working on panelization
Parts:
- D1: value (none) -> 1N4001
- R1: value (none) -> 4.7k
- turned D1 to 270 degrees
Connections:
- net +9V: now also D1.A; no longer D1.C
- net A: now also D1.C; no longer D1.A
Routing:
- net A: track 39.1 -> 40.1 mm
Changed lines of the file:
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@@
 <element name="SW2" library="mb_switches" package="3PDT" value="3PDT" x="12.7" y="8.89" smashed="yes"/>
 <element name="U$1" library="xc_library" package="BOARDLINK" value="BOARDLINK" x="9.906" y="19.685" smashed="yes"/>
-<element name="D1" library="mb_diodes" package="DO41-3" value="" x="23.018" y="5.743" smashed="yes" rot="R90">
-<attribute name="NAME" x="23.653" y="4.6508" size="1.27" layer="25" ratio="12" rot="R90"/>
-<attribute name="VALUE" x="25.812" y="3.838" size="1.27" layer="27" ratio="12" rot="R90"/>
+<element name="D1" library="mb_diodes" package="DO41-3" value="1N4001" x="22.982" y="5.757" smashed="yes" rot="R270">
+<attribute name="NAME" x="22.347" y="6.8492" size="1.27" layer="25" ratio="12" rot="R270"/>
+<attribute name="VALUE" x="20.188" y="7.662" size="1.27" layer="27" ratio="12" rot="R270"/>
 </element>
 <element name="+9V" library="mb_supply" package="SQUARE" value="+9V(T)" x="26.47" y="5.13" smashed="yes">
 <attribute name="NAME" x="28.805" y="3.44" size="1.016" layer="25" ratio="12" rot="R90"/>
 </element>
-<element name="R1" library="mb_resistors" package="R0207/3" value="" x="23" y="16" smashed="yes" rot="R270">
+<element name="R1" library="mb_resistors" package="R0207/3" value="4.7k" x="23" y="16" smashed="yes" rot="R270">
 <attribute name="NAME" x="22.365" y="17.27" size="1.27" layer="25" font="vector" ratio="12" rot="R270"/>
 <attribute name="VALUE" x="20.46" y="17.27" size="1.27" layer="27" font="vector" ratio="12" rot="R270"/>
@@
 <contactref element="U$1" pad="3"/>
 <contactref element="R1" pad="2"/>
-<wire x1="12.446" y1="19.685" x2="15.461" y2="22.7" width="0.4064" layer="1"/>
-<wire x1="27.8" y1="22.7" x2="28.5" y2="22" width="0.4064" layer="1"/>
-<wire x1="28.5" y1="22" x2="28.5" y2="9.5" width="0.4064" layer="1"/>
-<wire x1="27.5" y1="8.5" x2="28.5" y2="9.5" width="0.4064" layer="1"/>
-<wire x1="15.461" y1="22.7" x2="27.8" y2="22.7" width="0.4064" layer="1"/>
-<contactref element="D1" pad="A"/>
-<wire x1="23" y1="12.19" x2="23.018" y2="12.172" width="0.4064" layer="1"/>
-<wire x1="23.018" y1="12.172" x2="23.018" y2="9.553" width="0.4064" layer="1"/>
-<wire x1="23.018" y1="9.553" x2="24.071" y2="8.5" width="0.4064" layer="1"/>
-<wire x1="24.071" y1="8.5" x2="27.5" y2="8.5" width="0.4064" layer="1"/>
+<contactref element="D1" pad="C"/>
+<wire x1="24.549" y1="8" x2="22.982" y2="9.567" width="0.4064" layer="1"/>
+<wire x1="12.446" y1="19.685" x2="14.261" y2="21.5" width="0.4064" layer="1"/>
+<wire x1="21.27034375" y1="21.5" x2="21.942625" y2="22.17228125" width="0.4064" layer="1"/>
+<wire x1="21.942625" y1="22.17228125" x2="24.2" y2="22.17228125" width="0.4064" layer="1"/>
+<wire x1="24.2" y1="22.17228125" x2="24.72771875" y2="22.7" width="0.4064" layer="1"/>
+<wire x1="24.72771875" y1="22.7" x2="27.8" y2="22.7" width="0.4064" layer="1"/>
+<wire x1="27.8" y1="22.7" x2="28.4858" y2="22.0142" width="0.4064" layer="1"/>
+<wire x1="14.261" y1="21.5" x2="21.27034375" y2="21.5" width="0.4064" layer="1"/>
+<wire x1="23" y1="12.19" x2="23" y2="9.585" width="0.4064" layer="1"/>
+<wire x1="23" y1="9.585" x2="22.982" y2="9.567" width="0.4064" layer="1"/>
+<wire x1="28.4858" y1="22.0142" x2="28.4858" y2="8.4858" width="0.4064" layer="1"/>
+<wire x1="28.4858" y1="8.4858" x2="28" y2="8" width="0.4064" layer="1"/>
+<wire x1="28" y1="8" x2="24.549" y2="8" width="0.4064" layer="1"/>
 </signal>
 <signal name="N$7">
@@
 </signal>
 <signal name="+9V">
-<contactref element="D1" pad="C"/>
 <contactref element="+9V" pad="1"/>
-<wire x1="23.018" y1="1.933" x2="26.215" y2="5.13" width="0.4064" layer="1"/>
-<wire x1="26.215" y1="5.13" x2="26.47" y2="5.13" width="0.4064" layer="1"/>
+<contactref element="D1" pad="A"/>
+<wire x1="26.47" y1="5.13" x2="26.165" y2="5.13" width="0.4064" layer="1"/>
+<wire x1="26.165" y1="5.13" x2="22.982" y2="1.947" width="0.4064" layer="1"/>
 </signal>
 </signals>

Commit message: Commit Seeed board and backup files
Changed lines of the file:
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@@
 <element name="U$1" library="xc_library" package="BOARDLINK" value="BOARDLINK" x="9.906" y="19.685" smashed="yes"/>
 <element name="D1" library="mb_diodes" package="DO41-3" value="1N4001" x="22.982" y="5.757" smashed="yes" rot="R270">
-<attribute name="NAME" x="22.347" y="6.8492" size="1.27" layer="25" ratio="12" rot="R270"/>
-<attribute name="VALUE" x="20.188" y="7.662" size="1.27" layer="27" ratio="12" rot="R270"/>
+<attribute name="VALUE" x="22.588" y="6.762" size="0.6096" layer="27" ratio="12" rot="R270"/>
 </element>
 <element name="+9V" library="mb_supply" package="SQUARE" value="+9V(T)" x="26.47" y="5.13" smashed="yes">
@@
 </element>
 <element name="R1" library="mb_resistors" package="R0207/3" value="4.7k" x="23" y="16" smashed="yes" rot="R270">
-<attribute name="NAME" x="22.365" y="17.27" size="1.27" layer="25" font="vector" ratio="12" rot="R270"/>
-<attribute name="VALUE" x="20.46" y="17.27" size="1.27" layer="27" font="vector" ratio="12" rot="R270"/>
+<attribute name="VALUE" x="22.36" y="17.57" size="1.27" layer="27" font="vector" ratio="12" rot="R270"/>
 </element>
 <element name="D2" library="mb_diodes" package="LED3MM" value="LED3MM" x="26.95" y="11.6" smashed="yes" rot="R270"/>
